Commit message: add kinova gen3; gripper not configured

File: protos/6dof/urdf/combined_robot.urdf (robot description, URDF)
Before this commit: robot gen3_6dof_with_robotiq_2f_140, 22 links, 21 joints
Links:
- removed link base_link
- added link gen3_base_link, mass 1.697; collision mesh filename=package://kortex_description/arms/gen3/6dof/meshes/base_lin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; visual mesh filename=package://kortex_description/arms/gen3/6dof/meshes/base_lin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
Joints:
- joint joint_1: parent base_link -> gen3_base_link

File: resource/spot.urdf (robot description, URDF)
Before this commit: robot Spot, 78 links, 77 joints
Links:
- removed link SpotArm
- removed link spotarm_link1
- removed link spotarm_link2
- removed link spotarm_link3
- removed link spotarm_link4
- removed link spotarm_link5
- removed link spotarm_link6
- added link bicep_link, mass 1.262; collision mesh filename=package://kortex_description/arms/gen3/6dof/meshes/bicep_li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; visual mesh filename=package://kortex_description/arms/gen3/6dof/meshes/bicep_li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
- added link bracelet_link, mass 0.5; collision mesh filename=package://kortex_description/arms/gen3/6dof/meshes/bracelet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; visual mesh filename=package://kortex_description/arms/gen3/6dof/meshes/bracelet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
- added link camera_color_frame
- added link camera_depth_frame
- added link camera_link
- added link end_effector_link, mass 0
- added link forearm_link, mass 0.93; collision mesh filename=package://kortex_description/arms/gen3/6dof/meshes/forearm_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; visual mesh filename=package://kortex_description/arms/gen3/6dof/meshes/forearm_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
- added link gen3_base_link, mass 1.697; collision mesh filename=package://kortex_description/arms/gen3/6dof/meshes/base_lin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; visual mesh filename=package://kortex_description/arms/gen3/6dof/meshes/base_lin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
- added link left_inner_finger, mass 0.0104003125914103; collision mesh filename=package://robotiq_description/meshes/collision/2f_140/robot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; visual mesh filename=package://robotiq_description/meshes/visual/2f_140/robotiq_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
- added link left_inner_finger_pad; collision box size=0.03 0.07 0.0075; visual box size=0.027 0.065 0.0075
- added link left_inner_knuckle, mass 0.0271177346495152; collision mesh filename=package://robotiq_description/meshes/collision/2f_140/robot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; visual mesh filename=package://robotiq_description/meshes/visual/2f_140/robotiq_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
- added link left_outer_finger, mass 0.022614240507152; collision mesh filename=package://robotiq_description/meshes/collision/2f_140/robot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; visual mesh filename=package://robotiq_description/meshes/visual/2f_140/robotiq_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
- added link left_outer_knuckle, mass 0.00853198276973456; collision mesh filename=package://robotiq_description/meshes/collision/2f_140/robot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; visual mesh filename=package://robotiq_description/meshes/visual/2f_140/robotiq_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
- added link right_inner_finger, mass 0.0104003125914103; collision mesh filename=package://robotiq_description/meshes/collision/2f_140/robot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; visual mesh filename=package://robotiq_description/meshes/visual/2f_140/robotiq_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
- added link right_inner_finger_pad; collision box size=0.03 0.07 0.0075; visual box size=0.027 0.065 0.0075
- added link right_inner_knuckle, mass 0.0271177346495152; collision mesh filename=package://robotiq_description/meshes/collision/2f_140/robot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; visual mesh filename=package://robotiq_description/meshes/visual/2f_140/robotiq_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
- added link right_outer_finger, mass 0.022614240507152; collision mesh filename=package://robotiq_description/meshes/collision/2f_140/robot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; visual mesh filename=package://robotiq_description/meshes/visual/2f_140/robotiq_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
- added link right_outer_knuckle, mass 0.00853198276973456; collision mesh filename=package://robotiq_description/meshes/collision/2f_140/robot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; visual mesh filename=package://robotiq_description/meshes/visual/2f_140/robotiq_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
- added link robotiq_2f_base_link, mass 0.22652; collision mesh filename=package://robotiq_description/meshes/collision/2f_140/robot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; visual mesh filename=package://robotiq_description/meshes/visual/2f_140/robotiq_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
- added link shoulder_link, mass 1.377; collision mesh filename=package://kortex_description/arms/gen3/6dof/meshes/shoulder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; visual mesh filename=package://kortex_description/arms/gen3/6dof/meshes/shoulder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
- added link spherical_wrist_1_link, mass 0.6781; collision mesh filename=package://kortex_description/arms/gen3/6dof/meshes/spherica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; visual mesh filename=package://kortex_description/arms/gen3/6dof/meshes/spherica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
- added link spherical_wrist_2_link, mass 0.678; collision mesh filename=package://kortex_description/arms/gen3/6dof/meshes/spherica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; visual mesh filename=package://kortex_description/arms/gen3/6dof/meshes/spherica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
Joints:
- removed joint Slider11
- removed joint base_link_SpotArm_joint
- removed joint spotarm_1_joint
- removed joint spotarm_2_joint
- removed joint spotarm_3_joint
- removed joint spotarm_4_joint
- removed joint spotarm_5_joint
- removed joint spotarm_6_joint
- added joint arm_to_gripper_joint: type fixed, parent end_effector_link, child robotiq_2f_base_link, origin xyz=0 0 -0.01 rpy=0 0 -1.5708
- added joint base_link_to_front: type fixed, parent base_link, child front, origin xyz=0 0 0 rpy=0 0 0
- added joint base_link_to_gen3_base_link: type fixed, parent base_link, child gen3_base_link, origin xyz=0.256 0 0.1118 rpy=0.0 0.0 0.0
- added joint camera_module: type fixed, parent end_effector_link, child camera_link, origin xyz=0 0.05639 -0.00305 rpy=3.14159265358979 3.14159265358979 0
- added joint color_module: type fixed, parent end_effector_link, child camera_color_frame, origin xyz=0 0.05639 -0.00305 rpy=3.14159265358979 3.14159265358979 0
- added joint depth_module: type fixed, parent end_effector_link, child camera_depth_frame, origin xyz=0.0275 0.066 -0.00305 rpy=3.14159265358979 3.14159265358979 0
- added joint end_effector: type fixed, parent bracelet_link, child end_effector_link, origin xyz=0 0 -0.061525 rpy=3.1416 0 -3.1416, axis 0 0 0
- added joint finger_joint: type revolute, parent robotiq_2f_base_link, child left_outer_knuckle, origin xyz=0 -0.030601 0.054905 rpy=2.2957963267948966 0 0, axis -1 0 0, limit lower=0 upper=0.7 effort=1000 velocity=2.0
- added joint joint_1: type continuous, parent gen3_base_link, child shoulder_link, origin xyz=0 0 0.15643 rpy=-3.1416 0.0 0.0, axis 0 0 1, limit effort=39 velocity=1.3963
- added joint joint_2: type revolute, parent shoulder_link, child bicep_link, origin xyz=0 0.005375 -0.12838 rpy=1.5708 0.0 0.0, axis 0 0 1, limit lower=-2.24 upper=2.24 effort=39 velocity=1.3963
- added joint joint_3: type revolute, parent bicep_link, child forearm_link, origin xyz=0 -0.41 0 rpy=3.1416 0 0, axis 0 0 1, limit lower=-2.57 upper=2.57 effort=39 velocity=1.3963
- added joint joint_4: type continuous, parent forearm_link, child spherical_wrist_1_link, origin xyz=0 0.20843 -0.006375 rpy=1.5708 0.0 0.0, axis 0 0 1, limit effort=9 velocity=1.2218
- added joint joint_5: type revolute, parent spherical_wrist_1_link, child spherical_wrist_2_link, origin xyz=0 -0.00017505 -0.10593 rpy=-1.5708 0.0 0.0, axis 0 0 1, limit lower=-2.09 upper=2.09 effort=9 velocity=1.2218
- added joint joint_6: type continuous, parent spherical_wrist_2_link, child bracelet_link, origin xyz=0 0.10593 -0.00017505 rpy=1.5708 0.0 0.0, axis 0 0 1, limit effort=9 velocity=1.2218
- added joint left_inner_finger_joint: type revolute, parent left_outer_finger, child left_inner_finger, origin xyz=0 0.0817554015893473 -0.0282203446692936 rpy=-0.725 0 0, axis 1 0 0, limit lower=-0.8757 upper=0.8757 effort=1000 velocity=2.0, mimic joint=finger_joint multiplier=1 offset=0
- added joint left_inner_finger_pad_joint: type fixed, parent left_inner_finger, child left_inner_finger_pad, origin xyz=0 0.0457554015893473 -0.0272203446692936 rpy=0 0 0, axis 0 0 1
- added joint left_inner_knuckle_joint: type revolute, parent robotiq_2f_base_link, child left_inner_knuckle, origin xyz=0 -0.0127 0.06142 rpy=2.2957963267948966 0 0.0, axis 1 0 0, limit lower=-0.8757 upper=0.8757 effort=1000 velocity=2.0, mimic joint=finger_joint multiplier=-1 offset=0
- added joint left_outer_finger_joint: type fixed, parent left_outer_knuckle, child left_outer_finger, origin xyz=0 0.01821998610742 0.0260018192872234 rpy=0 0 0, axis 1 0 0
- added joint right_inner_finger_joint: type revolute, parent right_outer_finger, child right_inner_finger, origin xyz=0 0.0817554015893473 -0.0282203446692936 rpy=-0.725 0 0, axis 1 0 0, limit lower=-0.8757 upper=0.8757 effort=1000 velocity=2.0, mimic joint=finger_joint multiplier=1 offset=0
- added joint right_inner_finger_pad_joint: type fixed, parent right_inner_finger, child right_inner_finger_pad, origin xyz=0 0.0457554015893473 -0.0272203446692936 rpy=0 0 0, axis 0 0 1
- added joint right_inner_knuckle_joint: type revolute, parent robotiq_2f_base_link, child right_inner_knuckle, origin xyz=0 0.0127 0.06142 rpy=2.2957963267948966 0 -3.141592653589793, axis 1 0 0, limit lower=-0.8757 upper=0.8757 effort=1000 velocity=2.0, mimic joint=finger_joint multiplier=-1 offset=0
- added joint right_outer_finger_joint: type fixed, parent right_outer_knuckle, child right_outer_finger, origin xyz=0 0.01821998610742 0.0260018192872234 rpy=0 0 0, axis 1 0 0
- added joint right_outer_knuckle_joint: type revolute, parent robotiq_2f_base_link, child right_outer_knuckle, origin xyz=0 0.030601 0.054905 rpy=2.2957963267948966 0 3.141592653589793, axis 1 0 0, limit lower=-0.725 upper=0.725 effort=1000 velocity=2.0, mimic joint=finger_joint multiplier=-1 offset=0
