Commit message: gripper working correctly in rviz but not in webots

File: resource/spot.urdf (robot description, URDF)
Before this commit: robot Spot, 93 links, 92 joints
Joints:
- joint arm_to_gripper_joint: origin xyz=0 0 -0.01 rpy=0 0 -1.5708 -> xyz=0 0 -0.01 rpy=0 0 1.5708

Commit message: fixed moveit

File: resource/spot.urdf (robot description, URDF)
Before this commit: robot Spot, 93 links, 92 joints
Links:
- removed link gripper_centre
- removed link gripper_left_finger_link
- removed link gripper_right_finger_link
Joints:
- removed joint gripper_centre_joint
- removed joint gripper_left_finger_joint
- removed joint gripper_right_finger_joint

Commit message: fix moveit servo, gripper closing in webots simulation [WIP]

File: resource/spot.urdf (robot description, URDF)
Before this commit: robot Spot, 90 links, 89 joints
Joints:
- joint finger_joint: limit lower=0 upper=0.7 effort=1000 velocity=2.0 -> lower=0 upper=0.8 effort=1000 velocity=2.0
- joint joint_3: limit lower=-2.57 upper=2.57 effort=39 velocity=1.3963 -> lower=-3.2 upper=3.2 effort=39 velocity=1.3963
- joint right_outer_knuckle_joint: limit lower=-0.725 upper=0.725 effort=1000 velocity=2.0 -> lower=-0.8 upper=0.0 effort=1000 velocity=2.0

Commit message: clean spot sim for drl

File: resource/spot.urdf (robot description, URDF)
Before this commit: robot Spot, 78 links, 77 joints
Links:
- removed link SpotArm
- removed link cap screw
- removed link cap screw(1)
- removed link cap screw(10)
- removed link cap screw(11)
- removed link cap screw(12)
- removed link cap screw(13)
- removed link cap screw(14)
- removed link cap screw(15)
- removed link cap screw(16)
- removed link cap screw(17)
- removed link cap screw(18)
- removed link cap screw(19)
- removed link cap screw(2)
- removed link cap screw(3)
- removed link cap screw(4)
- removed link cap screw(5)
- removed link cap screw(6)
- removed link cap screw(7)
- removed link cap screw(8)
- removed link cap screw(9)
- removed link front
- removed link gripper_centre
- removed link gripper_left_finger_link
- removed link gripper_right_finger_link
- removed link kinect color
- removed link kinect range
- removed link spotarm_link1
- removed link spotarm_link2
- removed link spotarm_link3
- removed link spotarm_link4
- removed link spotarm_link5
- removed link spotarm_link6
Joints:
- removed joint Slider11
- removed joint base_link_SpotArm_joint
- removed joint front_cap screw(1)_joint
- removed joint front_cap screw(10)_joint
- removed joint front_cap screw(11)_joint
- removed joint front_cap screw(12)_joint
- removed joint front_cap screw(13)_joint
- removed joint front_cap screw(14)_joint
- removed joint front_cap screw(15)_joint
- removed joint front_cap screw(16)_joint
- removed joint front_cap screw(17)_joint
- removed joint front_cap screw(18)_joint
- removed joint front_cap screw(19)_joint
- removed joint front_cap screw(2)_joint
- removed joint front_cap screw(3)_joint
- removed joint front_cap screw(4)_joint
- removed joint front_cap screw(5)_joint
- removed joint front_cap screw(6)_joint
- removed joint front_cap screw(7)_joint
- removed joint front_cap screw(8)_joint
- removed joint front_cap screw(9)_joint
- removed joint front_cap screw_joint
- removed joint gripper_centre_joint
- removed joint gripper_left_finger_joint
- removed joint gripper_right_finger_joint
- removed joint solid_kinect color_joint
- removed joint solid_kinect range_joint
- removed joint spotarm_1_joint
- removed joint spotarm_2_joint
- removed joint spotarm_3_joint
- removed joint spotarm_4_joint
- removed joint spotarm_5_joint
- removed joint spotarm_6_joint

Commit message: add dex board detection

File: resource/spot.urdf (robot description, URDF)
Before this commit: robot Spot, 90 links, 89 joints
Joints:
- joint base_link_solid_joint: origin xyz=0.496831 0.000001 0.104801 rpy=1.2208 -0.00001 -1.570793 -> xyz=0.496831 0.000001 0.104801 rpy=0 0 0
- joint solid_kinect color_joint: origin xyz=0 0 -0.0127 rpy=-2.356193 1.570792 -0.7854 -> xyz=0 0 -0.0127 rpy=0 0 0
- joint solid_kinect range_joint: origin xyz=0 0 -0.0127 rpy=-0.785397 1.570792 0.785397 -> xyz=0 0 -0.0127 rpy=0 0 0

Commit message: fix moveit joint control

File: resource/spot.urdf (robot description, URDF)
Before this commit: robot Spot, 90 links, 89 joints
Joints:
- joint joint_1: limit effort=39 velocity=1.3963 -> lower=-3.2 upper=3.2 effort=39 velocity=1.3963; type continuous -> revolute
- joint joint_4: limit effort=9 velocity=1.2218 -> lower=-3.2 upper=3.2 effort=9 velocity=1.2218; type continuous -> revolute
- joint joint_6: limit effort=9 velocity=1.2218 -> lower=-3.2 upper=3.2 effort=9 velocity=1.2218; type continuous -> revolute

Commit message: save dexboard pose in yaml; fix kinova joint limits

File: resource/spot.urdf (robot description, URDF)
Before this commit: robot Spot, 90 links, 89 joints
Joints:
- joint joint_1: limit lower=-3.2 upper=3.2 effort=39 velocity=1.3963 -> lower=-6.3 upper=6.3 effort=39 velocity=1.3963
- joint joint_3: limit lower=-3.2 upper=3.2 effort=39 velocity=1.3963 -> lower=-6.3 upper=6.3 effort=39 velocity=1.3963
- joint joint_4: limit lower=-3.2 upper=3.2 effort=9 velocity=1.2218 -> lower=-6.3 upper=6.3 effort=9 velocity=1.2218
- joint joint_5: limit lower=-2.09 upper=2.09 effort=9 velocity=1.2218 -> lower=-2.23 upper=2.23 effort=9 velocity=1.2218
- joint joint_6: limit lower=-3.2 upper=3.2 effort=9 velocity=1.2218 -> lower=-6.3 upper=6.3 effort=9 velocity=1.2218
